Commit message: Compelete week2 assignment 1.

File: hrwros_ws/src/hrwros_assignments/hrwros_week2_assignment/urdf/hrwros_assignment1.xacro (robot description, xacro)
@@ -72,3 +72,11 @@
   </joint>
   <!-- Add your solution to assignment 1 here -->
+  <!-- bin 2-->
+  <xacro:include filename="$(find hrwros_support)/urdf/bin/bin.urdf.xacro"/>
+  <xacro:bin_urdf prefix="bin_2_"/>
+  <joint name="bin_2_joint" type="fixed">
+    <parent link="world_interface" />
+    <child link="bin_2_base_link" />
+    <origin xyz="2.5 1.8 0.0" rpy="0 0 0" />
+  </joint>
 </robot>
