Commit message: Complete week2 assignment 2

File: hrwros_ws/src/hrwros_assignments/hrwros_week2_assignment/urdf/hrwros_assignment2.xacro (robot description, xacro)
@@ -72,3 +72,19 @@
   </joint>
   <!-- Add your solution to assignment 2 here -->
+  <link name="sphere_1_link">
+    <visual>
+      <origin xyz="0 0 0.4" />
+      <geometry>
+        <sphere radius="0.4" />
+      </geometry>
+      <material name="spehere_1_color">
+        <color rgba="0 ${110/255} 0 1" />
+      </material>
+    </visual>
+  </link>
+  <joint name="shpere_1_joint" type="fixed">
+    <origin xyz="5.8 -5 0" />
+    <parent link="world" />
+    <child link="sphere_1_link" />
+  </joint>
 </robot>
