Commit message: Complete week2 assignment 3

File: hrwros_ws/src/hrwros_assignments/hrwros_week2_assignment/urdf/hrwros_assignment3.xacro (robot description, xacro)
@@ -65,10 +65,10 @@
   </joint>
   <!-- Update the below block for assignment 3 here -->
-  <xacro:include filename="$(find ur_description)/urdf/inc/ur5_macro.xacro"/>
-  <xacro:ur5_robot prefix="robot2_" safety_limits="true"/>
+  <xacro:include filename="$(find hrwros_week2_assignment)/urdf/robot/lrmate200ic_macro.xacro"/>
+  <xacro:fanuc_lrmate200ic prefix="robot2_" joint_limited="true"/>
   <joint name="robot2-robot2_pedestal_joint" type="fixed">
     <parent link="robot2_pedestal_link" />
     <child link="robot2_base_link" />
-    <origin xyz="0 0 0.6" rpy="0 0 ${radians(90)}" />
+    <origin xyz="-0.025 0 0.6" rpy="0 0 ${radians(180)}" />
   </joint>
 </robot>
