Commit message: Migrate week2 assignment1 to ros2.

File: hrwros_ws/src/hrwros/hrwros_support/urdf/ur.urdf.xacro (robot description, xacro)
@@ -45,5 +45,5 @@
     <xacro:arg name="simulation_controllers" default="" />
     <!-- initial position for simulations (Fake Hardware, Gazebo, Ignition) -->
-    <xacro:arg name="initial_positions_file" default="$(find ur_description)/config/initial_positions.yaml"/>
+    <xacro:arg name="initial_positions_file" default="$(find hrwros_support)/config/$(arg prefix)initial_positions.yaml"/>
     <!-- convert to property to use substitution in function -->
     <xacro:property name="initial_positions_file" default="$(arg initial_positions_file)"/>

File: hrwros_ws/src/hrwros_assignments/hrwros_week2_assignment/urdf/hrwros_assignment1.xacro (robot description, xacro)
@@ -12,6 +12,7 @@
   </xacro:robot_pedestal_urdf>
   <!-- Robot1 -->
-  <xacro:include filename="$(find ur_description)/urdf/inc/ur10_macro.xacro"/>
-  <xacro:ur10_robot prefix="robot1_" safety_limits="true"/>
+  <xacro:include filename="$(find hrwros_support)/urdf/ur.urdf.xacro" />
+  <xacro:simple_ur_robot name="robot1" ur_type="ur10" prefix="robot1_" parent="robot1_parent_link" safety_limits="true" />
+  <link name="robot1_parent_link" />
   <!-- Vacuum Gripper1 -->
   <xacro:include filename="$(find hrwros_support)/urdf/vacuum_gripper/vacuum_gripper.urdf.xacro"/>
@@ -35,5 +36,5 @@
   <origin xyz="0 0 0.95" rpy="0 0 0" />
   <parent link="robot1_pedestal_link" />
-  <child link="robot1_base_link" />
+  <child link="robot1_parent_link" />
   </joint>
   <!-- gripper1 to robot1. -->
@@ -64,9 +65,11 @@
     <child link="robot2_pedestal_link" />
   </joint>
-  <xacro:include filename="$(find ur_description)/urdf/inc/ur5_macro.xacro"/>
-  <xacro:ur5_robot prefix="robot2_" safety_limits="true"/>
+  <!-- Robot2 -->
+  <xacro:include filename="$(find hrwros_support)/urdf/ur.urdf.xacro" />
+  <xacro:simple_ur_robot name="robot1" ur_type="ur5" prefix="robot2_" parent="robot2_parent_link" safety_limits="true" />
+  <link name="robot2_parent_link" />
   <joint name="robot2-robot2_pedestal_joint" type="fixed">
     <parent link="robot2_pedestal_link" />
-    <child link="robot2_base_link" />
+    <child link="robot2_parent_link" />
     <origin xyz="0 0 0.6" rpy="0 0 ${radians(90)}" />
   </joint>

Commit message: Update assignment1.

File: hrwros_ws/src/hrwros/hrwros_support/urdf/ur.urdf.xacro (robot description, xacro)
@@ -3,107 +3,26 @@
   <!-- import main macro -->
   <xacro:include filename="$(find ur_description)/urdf/ur_macro.xacro"/>
-  <xacro:macro name="simple_ur_robot" params="name:='ur' ur_type prefix parent:='' safety_limits:=false">
-    <!-- robot name parameter -->
-    <xacro:arg name="name" default="${name}"/>
-    <!-- possible 'ur_type' values: ur3, ur3e, ur5, ur5e, ur10, ur10e, ur16e -->
-    <!-- the default value should raise an error in case this was called without defining the type -->
-    <xacro:arg name="ur_type" default="${ur_type}"/>
-    <!-- parameters -->
-    <xacro:arg name="prefix" default="${prefix}" />
-    <xacro:arg name="parent" default="${parent}"/>
-    <xacro:arg name="joint_limit_params" default="$(find ur_description)/config/$(arg ur_type)/joint_limits.yaml"/>
-    <xacro:arg name="kinematics_params" default="$(find ur_description)/config/$(arg ur_type)/default_kinematics.yaml"/>
-    <xacro:arg name="physical_params" default="$(find ur_description)/config/$(arg ur_type)/physical_parameters.yaml"/>
-    <xacro:arg name="visual_params" default="$(find ur_description)/config/$(arg ur_type)/visual_parameters.yaml"/>
-    <xacro:arg name="transmission_hw_interface" default=""/>
-    <xacro:arg name="safety_limits" default="${str(safety_limits)}"/>
-    <xacro:arg name="safety_pos_margin" default="0.15"/>
-    <xacro:arg name="safety_k_position" default="20"/>
-    <!-- ros2_control related parameters -->
-    <xacro:arg name="headless_mode" default="false" />
-    <xacro:arg name="robot_ip" default="0.0.0.0" />
-    <xacro:arg name="script_filename" default=""/>
-    <xacro:arg name="output_recipe_filename" default=""/>
-    <xacro:arg name="input_recipe_filename" default=""/>
-    <xacro:arg name="reverse_ip" default="0.0.0.0"/>
-    <xacro:arg name="script_command_port" default="50004"/>
-    <!--   tool communication related parameters-->
-    <xacro:arg name="use_tool_communication" default="false" />
-    <xacro:arg name="tool_voltage" default="0" />
-    <xacro:arg name="tool_parity" default="0" />
-    <xacro:arg name="tool_baud_rate" default="115200" />
-    <xacro:arg name="tool_stop_bits" default="1" />
-    <xacro:arg name="tool_rx_idle_chars" default="1.5" />
-    <xacro:arg name="tool_tx_idle_chars" default="3.5" />
-    <xacro:arg name="tool_device_name" default="/tmp/ttyUR" />
-    <xacro:arg name="tool_tcp_port" default="54321" />
-    <!-- Simulation parameters -->
-    <xacro:arg name="use_fake_hardware" default="false" />
-    <xacro:arg name="fake_sensor_commands" default="false" />
-    <xacro:arg name="sim_gazebo" default="false" />
-    <xacro:arg name="sim_ignition" default="false" />
-    <xacro:arg name="simulation_controllers" default="" />
-    <!-- initial position for simulations (Fake Hardware, Gazebo, Ignition) -->
-    <xacro:arg name="initial_positions_file" default="$(find hrwros_support)/config/$(arg prefix)initial_positions.yaml"/>
-    <!-- convert to property to use substitution in function -->
-    <xacro:property name="initial_positions_file" default="$(arg initial_positions_file)"/>
-    <!-- arm -->
+  <xacro:macro name="simple_ur_robot" params="ur_type name:='ur' prefix:='' parent:='' *origin safety_limits:=false ">
+    <xacro:property name="joint_limit_params" default="$(find ur_description)/config/${ur_type}/joint_limits.yaml"/>
+    <xacro:property name="kinematics_params" default="$(find ur_description)/config/${ur_type}/default_kinematics.yaml"/>
+    <xacro:property name="physical_params" default="$(find ur_description)/config/${ur_type}/physical_parameters.yaml"/>
+    <xacro:property name="visual_params" default="$(find ur_description)/config/${ur_type}/visual_parameters.yaml"/>
+    <xacro:property name="initial_positions_file" default="$(find hrwros_support)/config/${prefix}initial_positions.yaml"/>
     <xacro:ur_robot
-     name="$(arg name)"
-     prefix="$(arg prefix)"
-     parent="$(arg parent)"
-     joint_limits_parameters_file="$(arg joint_limit_params)"
-     kinematics_parameters_file="$(arg kinematics_params)"
-     physical_parameters_file="$(arg physical_params)"
-     visual_parameters_file="$(arg visual_params)"
-     transmission_hw_interface="$(arg transmission_hw_interface)"
-     safety_limits="$(arg safety_limits)"
-     safety_pos_margin="$(arg safety_pos_margin)"
-     safety_k_position="$(arg safety_k_position)"
-     use_fake_hardware="$(arg use_fake_hardware)"
-     fake_sensor_commands="$(arg fake_sensor_commands)"
-     sim_gazebo="$(arg sim_gazebo)"
-     sim_ignition="$(arg sim_ignition)"
-     headless_mode="$(arg headless_mode)"
+     name="${name}"
+     prefix="${prefix}"
+     parent="${parent}"
+     joint_limits_parameters_file="${joint_limit_params}"
+     kinematics_parameters_file="${kinematics_params}"
+     physical_parameters_file="${physical_params}"
+     visual_parameters_file="${visual_params}"
+     transmission_hw_interface=""
+     safety_limits="${str(safety_limits)}"
      initial_positions="${xacro.load_yaml(initial_positions_file)}"
-     use_tool_communication="$(arg use_tool_communication)"
-     tool_voltage="$(arg tool_voltage)"
-     tool_parity="$(arg tool_parity)"
-     tool_baud_rate="$(arg tool_baud_rate)"
-     tool_stop_bits="$(arg tool_stop_bits)"
-     tool_rx_idle_chars="$(arg tool_rx_idle_chars)"
-     tool_tx_idle_chars="$(arg tool_tx_idle_chars)"
-     tool_device_name="$(arg tool_device_name)"
-     tool_tcp_port="$(arg tool_tcp_port)"
-     robot_ip="$(arg robot_ip)"
-     script_filename="$(arg script_filename)"
-     output_recipe_filename="$(arg output_recipe_filename)"
-     input_recipe_filename="$(arg input_recipe_filename)"
-     reverse_ip="$(arg reverse_ip)"
-     script_command_port="$(arg script_command_port)">
-      <origin xyz="0 0 0" rpy="0 0 0" />
-      <!-- position robot in the world -->
+     script_filename=""
+     output_recipe_filename=""
+     input_recipe_filename="">
+      <xacro:insert_block name="origin" />
     </xacro:ur_robot>
-    <xacro:if value="$(arg sim_gazebo)">
-      <!-- Gazebo plugins -->
-      <gazebo reference="world">
-      </gazebo>
-      <gazebo>
-        <plugin filename="libgazebo_ros2_control.so" name="gazebo_ros2_control">
-          <parameters>$(arg simulation_controllers)</parameters>
-        </plugin>
-      </gazebo>
-    </xacro:if>
-    <xacro:if value="$(arg sim_ignition)">
-      <!-- Gazebo plugins -->
-      <gazebo reference="world">
-      </gazebo>
-      <gazebo>
-        <plugin filename="libign_ros2_control-system.so" name="ign_ros2_control::IgnitionROS2ControlPlugin">
-          <parameters>$(arg simulation_controllers)</parameters>
-          <controller_manager_node_name>$(arg prefix)controller_manager</controller_manager_node_name>
-        </plugin>
-      </gazebo>
-    </xacro:if>
   </xacro:macro>
 </robot>

File: hrwros_ws/src/hrwros_assignments/hrwros_week2_assignment/urdf/hrwros_assignment1.xacro (robot description, xacro)
@@ -9,10 +9,12 @@
   <xacro:include filename="$(find hrwros_support)/urdf/robot_pedestal/robot_pedestal.urdf.xacro"/>
   <xacro:robot_pedestal_urdf pedestal_prefix="robot1_" pedestal_parent="world_interface" pedestal_height="0.95">
+    <!-- robot1 to pedestal. -->
     <origin xyz="0.5 1.8 0.0" rpy="0 0 0"/>
   </xacro:robot_pedestal_urdf>
   <!-- Robot1 -->
   <xacro:include filename="$(find hrwros_support)/urdf/ur.urdf.xacro" />
-  <xacro:simple_ur_robot name="robot1" ur_type="ur10" prefix="robot1_" parent="robot1_parent_link" safety_limits="true" />
-  <link name="robot1_parent_link" />
+  <xacro:simple_ur_robot name="robot1" ur_type="ur10" prefix="robot1_" parent="robot1_pedestal_link" safety_limits="true">
+    <origin xyz="0 0 0.95" rpy="0 0 0" />
+  </xacro:simple_ur_robot>
   <!-- Vacuum Gripper1 -->
   <xacro:include filename="$(find hrwros_support)/urdf/vacuum_gripper/vacuum_gripper.urdf.xacro"/>
@@ -31,10 +33,4 @@
     <child link="robot1_pedestal_link" />
     <origin xyz="0.5 1.8 0.0" rpy="0.0 0.0 0.0"/>
-  </joint>
-  <!-- robot1 to pedestal. -->
-  <joint name="robot1_to_pedestal" type="fixed">
-  <origin xyz="0 0 0.95" rpy="0 0 0" />
-  <parent link="robot1_pedestal_link" />
-  <child link="robot1_parent_link" />
   </joint>
   <!-- gripper1 to robot1. -->
@@ -66,12 +62,7 @@
   </joint>
   <!-- Robot2 -->
-  <xacro:include filename="$(find hrwros_support)/urdf/ur.urdf.xacro" />
-  <xacro:simple_ur_robot name="robot1" ur_type="ur5" prefix="robot2_" parent="robot2_parent_link" safety_limits="true" />
-  <link name="robot2_parent_link" />
-  <joint name="robot2-robot2_pedestal_joint" type="fixed">
-    <parent link="robot2_pedestal_link" />
-    <child link="robot2_parent_link" />
+  <xacro:simple_ur_robot name="robot2" ur_type="ur5" prefix="robot2_" parent="robot2_pedestal_link" safety_limits="true">
     <origin xyz="0 0 0.6" rpy="0 0 ${radians(90)}" />
-  </joint>
+  </xacro:simple_ur_robot>
   <!-- Add your solution to assignment 1 here -->
   <!-- bin 2-->

Commit message: Fix rivz config & initial ros param.

File: hrwros_ws/src/hrwros/hrwros_support/urdf/ur.urdf.xacro (robot description, xacro)
@@ -8,5 +8,5 @@
     <xacro:property name="physical_params" default="$(find ur_description)/config/${ur_type}/physical_parameters.yaml"/>
     <xacro:property name="visual_params" default="$(find ur_description)/config/${ur_type}/visual_parameters.yaml"/>
-    <xacro:property name="initial_positions_file" default="$(find hrwros_support)/config/${prefix}initial_positions.yaml"/>
+    <xacro:property name="initial_positions_file" default="$(find ur_description)/config/initial_positions.yaml"/>
     <xacro:ur_robot
      name="${name}"

File: hrwros_ws/src/hrwros_assignments/hrwros_week2_assignment/urdf/hrwros_assignment2.xacro (robot description, xacro)
@@ -12,6 +12,8 @@
   </xacro:robot_pedestal_urdf>
   <!-- Robot1 -->
-  <xacro:include filename="$(find ur_description)/urdf/inc/ur10_macro.xacro"/>
-  <xacro:ur10_robot prefix="robot1_" safety_limits="true"/>
+  <xacro:include filename="$(find hrwros_support)/urdf/ur.urdf.xacro" />
+  <xacro:simple_ur_robot name="robot1" ur_type="ur10" prefix="robot1_" parent="robot1_pedestal_link" safety_limits="true">
+    <origin xyz="0 0 0.95" rpy="0 0 0" />
+  </xacro:simple_ur_robot>
   <!-- Vacuum Gripper1 -->
   <xacro:include filename="$(find hrwros_support)/urdf/vacuum_gripper/vacuum_gripper.urdf.xacro"/>
@@ -30,10 +32,4 @@
     <child link="robot1_pedestal_link" />
     <origin xyz="0.5 1.8 0.0" rpy="0.0 0.0 0.0"/>
-  </joint>
-  <!-- robot1 to pedestal. -->
-  <joint name="robot1_to_pedestal" type="fixed">
-  <origin xyz="0 0 0.95" rpy="0 0 0" />
-  <parent link="robot1_pedestal_link" />
-  <child link="robot1_base_link" />
   </joint>
   <!-- gripper1 to robot1. -->
@@ -64,11 +60,8 @@
     <child link="robot2_pedestal_link" />
   </joint>
-  <xacro:include filename="$(find ur_description)/urdf/inc/ur5_macro.xacro"/>
-  <xacro:ur5_robot prefix="robot2_" safety_limits="true"/>
-  <joint name="robot2-robot2_pedestal_joint" type="fixed">
-    <parent link="robot2_pedestal_link" />
-    <child link="robot2_base_link" />
+  <!-- Robot2 -->
+  <xacro:simple_ur_robot name="robot2" ur_type="ur5" prefix="robot2_" parent="robot2_pedestal_link" safety_limits="true">
     <origin xyz="0 0 0.6" rpy="0 0 ${radians(90)}" />
-  </joint>
+  </xacro:simple_ur_robot>
   <!-- Add your solution to assignment 2 here -->
   <link name="sphere_1_link">

File: hrwros_ws/src/hrwros_assignments/hrwros_week2_assignment/urdf/hrwros_assignment3.xacro (robot description, xacro)
@@ -12,6 +12,8 @@
   </xacro:robot_pedestal_urdf>
   <!-- Robot1 -->
-  <xacro:include filename="$(find ur_description)/urdf/inc/ur10_macro.xacro"/>
-  <xacro:ur10_robot prefix="robot1_" safety_limits="true"/>
+  <xacro:include filename="$(find hrwros_support)/urdf/ur.urdf.xacro" />
+  <xacro:simple_ur_robot name="robot1" ur_type="ur10" prefix="robot1_" parent="robot1_pedestal_link" safety_limits="true">
+    <origin xyz="0 0 0.95" rpy="0 0 0" />
+  </xacro:simple_ur_robot>
   <!-- Vacuum Gripper1 -->
   <xacro:include filename="$(find hrwros_support)/urdf/vacuum_gripper/vacuum_gripper.urdf.xacro"/>

File: hrwros_ws/src/hrwros_assignments/hrwros_week2_assignment/urdf/robot/lrmate200ic_macro.xacro (robot description, xacro)
@@ -4,5 +4,5 @@
   <!-- NOTE: joint_limited is not used in this file -->
   <xacro:macro name="fanuc_lrmate200ic" params="prefix joint_limited:=false">
-    <!-- links: main serial chain -->
+    <!-- links main serial chain -->
     <link name="${prefix}base_link">
       <visual>
@@ -110,5 +110,5 @@
       </collision>
     </link>
-    <!-- joints: main serial chain -->
+    <!-- joints main serial chain -->
     <joint name="${prefix}joint_1" type="revolute">
       <origin xyz="0 0 0.330" rpy="0 0 0" />
@@ -153,5 +153,5 @@
       <limit effort="0" lower="-6.2832" upper="6.2832" velocity="12.5664" />
     </joint>
-    <!-- ROS-Industrial 'base' frame: base_link to Fanuc World Coordinates transform -->
+    <!-- ROS-Industrial 'base' frame base_link to Fanuc World Coordinates transform -->
     <link name="${prefix}base" />
     <joint name="${prefix}base_link-base" type="fixed">
@@ -160,5 +160,5 @@
       <child link="${prefix}base"/>
     </joint>
-    <!-- ROS-Industrial 'flange' frame: attachment point for EEF models -->
+    <!-- ROS-Industrial 'flange' frame attachment point for EEF models -->
     <link name="${prefix}flange" />
     <joint name="${prefix}joint_6-flange" type="fixed">
@@ -167,5 +167,5 @@
       <child link="${prefix}flange" />
     </joint>
-    <!-- ROS-Industrial 'tool0' frame: all-zeros tool frame -->
+    <!-- ROS-Industrial 'tool0' frame all-zeros tool frame -->
     <link name="${prefix}tool0" />
     <joint name="${prefix}link_6-tool0" type="fixed">
